Commit message: Updated README with solution to ros control not finding controller manager

File: src/racecar_description/urdf/racecar.xacro (robot description, xacro)
@@ -41,5 +41,5 @@
       <material name="black" />
     </visual>
-    <collision>robot
+    <collision>
       <xacro:left_wheels_collision_geometry />
     </collision>
